Commit message: Added camera

File: description/common_properties.xacro (robot description, xacro)
@@ -12,4 +12,7 @@
     <material name="black">
         <color rgba="0 0 0 1" />
+    </material>
+    <material name="red">
+        <color rgba="1 0 0 1" />
     </material>
     <!-- Specify some standard inertial calculations https://en.wikipedia.org/wiki/List_of_moments_of_inertia -->

File: description/lidar.xacro (robot description, xacro)
@@ -24,5 +24,5 @@
         <origin xyz="0.05 0 0.17" rpy="0 0 0" />
     </joint>
-    <!-- <gazebo reference="lidar_link">
+    <gazebo reference="lidar_link">
         <sensor name='laser' type='gpu_lidar'>
             <pose>0 0 0 0 0 0</pose>
@@ -43,36 +43,5 @@
             </lidar>
             <topic>lidar</topic>
-            <gz_frame_id>lidar_link</gz_frame_id>
-        </sensor>
-    </gazebo> -->
-    <gazebo reference="lidar_link">
-        <sensor name='gpu_lidar' type='gpu_lidar'>"
-            <pose>0 0 0 0 0 0</pose>
-            <topic>lidar</topic>
-            <update_rate>10</update_rate>
-            <ray>
-                <scan>
-                    <horizontal>
-                        <samples>640</samples>
-                        <resolution>1</resolution>
-                        <min_angle>-1.396263</min_angle>
-                        <max_angle>1.396263</max_angle>
-                    </horizontal>
-                    <vertical>
-                        <samples>1</samples>
-                        <resolution>0.01</resolution>
-                        <min_angle>0</min_angle>
-                        <max_angle>0</max_angle>
-                    </vertical>
-                </scan>
-                <range>
-                    <min>0.08</min>
-                    <max>10.0</max>
-                    <resolution>0.01</resolution>
-                </range>
-            </ray>
-            <always_on>1</always_on>
-            <visualize>true</visualize>
-            <gz_frame_id>lidar_link</gz_frame_id>
+              <gz_frame_id>lidar_link</gz_frame_id>
         </sensor>
     </gazebo>

File: description/robot.urdf.xacro (robot description, xacro)
@@ -5,3 +5,4 @@
     <xacro:include filename="robot_gazebo.xacro" />
     <xacro:include filename="lidar.xacro" />
+    <xacro:include filename="camera.xacro" />
 </robot>
